File: pcb/zenith.kicad_sch (KiCad schematic)
At the start: 0 parts

Commit message: pcb: initial schematic + pcb
Parts:
- added CM1: RX5808, lcsc:COMM-SMD_12P_RX5808, symbol lcsc:RX5808
- added J1: Conn_01x04_Pin, Connector_PinHeader_2.54mm:PinHeader_1x04_P2.54mm_Vertical, symbol Connector:Conn_01x04_Pin
- added J2: Conn_Coaxial, Connector_Coaxial:SMA_Amphenol_901-144_Vertical, symbol Connector:Conn_Coaxial
- added J3: Conn_Coaxial_x2, Connector_Coaxial:BNC_Win_364A2x95_Horizontal, symbol Connector:Conn_Coaxial_x2
- added R1: 100k, Resistor_THT:R_Axial_DIN0204_L3.6mm_D1.6mm_P7.62mm_Horizontal, symbol Device:R
- added SW1, SW2: SW_Push, Button_Switch_THT:SW_PUSH_6mm, symbol Switch:SW_Push
- added U2: XIAO-RP2040-DIP, XIAO_PCB:XIAO-RP2040-DIP, symbol Seeed_Studio_XIAO_Series:XIAO-RP2040-DIP
Connections:
- new net +3.3V: J1.1 (Pin_1), U2.12 (3V3)
- new net +5V: CM1.8 (+5V), U2.14 (VBUS)
- new net ANT: CM1.2 (ANT), J2.1 (In)
- new net AUDIO: CM1.10 (A6.5M), J3.2 (IN2)
- new net BTN1: SW1.1, U2.10 (GPIO4/MISO)
- new net BTN2: SW2.1, U2.7 (GPIO0/TX)
- new net GND: CM1.1 (GND), CM1.12 (GND), CM1.3 (GND), CM1.7 (GND), J1.2 (Pin_2), J2.2 (Ext), J3.3 (EXT), R1.1, SW1.2, SW2.2, U2.13 (GND)
- new net MOSI: CM1.4 (CH1), U2.11 (GPIO3/MOSI)
- new net RSSI: CM1.9 (RSSI), R1.2, U2.1 (GPIO26/ADC0/A0)
- new net RX_CS: CM1.5 (CH2), U2.8 (GPIO1/RX)
- new net SCK: CM1.6 (CH3), U2.9 (GPIO2/SCK)
- new net SCL: J1.3 (Pin_3), U2.6 (GPIO7/SCL)
- new net SDA: J1.4 (Pin_4), U2.5 (GPIO6/SDA)
- new net VIDEO: CM1.11 (VIDEO), J3.1 (IN1)
Other:
- note added: "Buttons"
- note added: "Microcontroller"
- note added: "OLED Module"
- note added: "RCA Outputs"
- note added: "RX Module"
- note added: "SMA Antenna"
